File: Hardware/Driver.brd (EAGLE design)
At the start: 50 x 22.5 mm, 58 parts, among them IC1 STM32F303CBT, IC2 78L12F, IC3 78L33, IC4 RT9629, Q1 PSMN, Q2 PSMN, Q3 PSMN, Q4 PSMN, Q5 PSMN, Q6 PSMN

Commit message: Dimensioning R + C
Parts:
- C1, C3, C5, C6, C7, C8: value (none) -> 100n
- C10, C9: value (none) -> 10u
- C11, C16, C17, C18: value (none) -> 1n
- C12: value (none) -> 22p
- C13, C14, C15: value (none) -> 1u
- R1: value (none) -> 10k
- R10, R11, R12, R2: value (none) -> 4k7
- R13, R14, R15, R3, R5, R6: value (none) -> 1k
- R4: value VISHAY_WSK1216 -> R001
- R7, R8: value (none) -> 100k
- R9: value (none) -> 51k
